Commit message: final submission

File: Assets/abb120/urdf/abb.xacro (robot description, xacro)
@@ -144,4 +144,84 @@
   </collision>
 </link>
+<link name="left_gripper_1">
+  <inertial>
+    <origin xyz="-0.6134605599811394 0.0001383187190899804 -0.3982785134737753" rpy="0 0 0"/>
+    <mass value="0.0035451260308642795"/>
+    <inertia ixx="0.0" iyy="0.0" izz="0.0" ixy="0.0" iyz="-0.0" ixz="0.0"/>
+  </inertial>
+  <visual>
+    <origin xyz="-0.627956 -0.627706 -0.810557" rpy="0 0 0"/>
+    <geometry>
+      <mesh filename="package://meshes/left_gripper_1.stl" scale="0.001 0.001 0.001"/>
+    </geometry>
+    <material name="silver"/>
+  </visual>
+  <collision>
+    <origin xyz="-0.627956 -0.627706 -0.810557" rpy="0 0 0"/>
+    <geometry>
+      <mesh filename="package://meshes/left_gripper_1.stl" scale="0.001 0.001 0.001"/>
+    </geometry>
+  </collision>
+</link>
+<link name="right_gripper_1">
+  <inertial>
+    <origin xyz="-0.6423416065798675 0.0001492846021573513 -0.3982746545264991" rpy="0 0 0"/>
+    <mass value="0.0035451260306269467"/>
+    <inertia ixx="0.0" iyy="0.0" izz="0.0" ixy="0.0" iyz="-0.0" ixz="-0.0"/>
+  </inertial>
+  <visual>
+    <origin xyz="-0.627956 -0.627706 -0.810557" rpy="0 0 0"/>
+    <geometry>
+      <mesh filename="package://meshes/right_gripper_1.stl" scale="0.001 0.001 0.001"/>
+    </geometry>
+    <material name="silver"/>
+  </visual>
+  <collision>
+    <origin xyz="-0.627956 -0.627706 -0.810557" rpy="0 0 0"/>
+    <geometry>
+      <mesh filename="package://meshes/right_gripper_1.stl" scale="0.001 0.001 0.001"/>
+    </geometry>
+  </collision>
+</link>
+<link name="camera_1">
+  <inertial>
+    <origin xyz="9.342563472479823e-06 0.01270209988539206 0.004959021796750063" rpy="0 0 0"/>
+    <mass value="0.2998999503460273"/>
+    <inertia ixx="0.000116" iyy="0.000116" izz="3e-05" ixy="-0.0" iyz="-0.0" ixz="-0.0"/>
+  </inertial>
+  <visual>
+    <origin xyz="-7e-05 -0.668805 -0.293055" rpy="0 0 0"/>
+    <geometry>
+      <mesh filename="package://meshes/camera_1.stl" scale="0.001 0.001 0.001"/>
+    </geometry>
+    <material name="silver"/>
+  </visual>
+  <collision>
+    <origin xyz="-7e-05 -0.668805 -0.293055" rpy="0 0 0"/>
+    <geometry>
+      <mesh filename="package://meshes/camera_1.stl" scale="0.001 0.001 0.001"/>
+    </geometry>
+  </collision>
+</link>
+<link name="ef_body_1">
+  <inertial>
+    <origin xyz="6.411121603684631e-06 1.1494758027863483e-05 0.020963560953154603" rpy="0 0 0"/>
+    <mass value="0.10781653983510255"/>
+    <inertia ixx="2e-05" iyy="2.2e-05" izz="7e-06" ixy="0.0" iyz="-0.0" ixz="0.0"/>
+  </inertial>
+  <visual>
+    <origin xyz="-4.9e-05 -0.627833 -0.36807" rpy="0 0 0"/>
+    <geometry>
+      <mesh filename="package://meshes/ef_body_1.stl" scale="0.001 0.001 0.001"/>
+    </geometry>
+    <material name="silver"/>
+  </visual>
+  <collision>
+    <origin xyz="-4.9e-05 -0.627833 -0.36807" rpy="0 0 0"/>
+    <geometry>
+      <mesh filename="package://meshes/ef_body_1.stl" scale="0.001 0.001 0.001"/>
+    </geometry>
+  </collision>
+</link>
 <joint name="Revolute 1" type="continuous">
   <origin xyz="0.0 0.166 0.0" rpy="0 0 0"/>
@@ -180,3 +260,23 @@
   <axis xyz="0.000134 0.000374 1.0"/>
 </joint>
+<joint name="Rigid 8" type="fixed">
+  <origin xyz="0.627907 -0.000127 0.442487" rpy="0 0 0"/>
+  <parent link="ef_body_1"/>
+  <child link="left_gripper_1"/>
+</joint>
+<joint name="Rigid 9" type="fixed">
+  <origin xyz="0.627907 -0.000127 0.442487" rpy="0 0 0"/>
+  <parent link="ef_body_1"/>
+  <child link="right_gripper_1"/>
+</joint>
+<joint name="Rigid 10" type="fixed">
+  <origin xyz="0.03103 0.040973 -0.00902" rpy="0 0 0"/>
+  <parent link="link_five_1"/>
+  <child link="camera_1"/>
+</joint>
+<joint name="Rigid 11" type="fixed">
+  <origin xyz="1e-06 2e-06 0.007" rpy="0 0 0"/>
+  <parent link="link_six_1"/>
+  <child link="ef_body_1"/>
+</joint>
 </robot>

File: Assets/abb120/urdf/abb120.urdf (robot description, URDF)
Before this commit: robot abb, 7 links, 6 joints
Links:
- added link camera_1, mass 0.2998999503460273; collision mesh filename=package://meshes/camera_1.stl scale=0.001 0.001 0.001; visual mesh filename=package://meshes/camera_1.stl scale=0.001 0.001 0.001
- added link ef_body_1, mass 0.10781653983510255; collision mesh filename=package://meshes/ef_body_1.stl scale=0.001 0.001 0.001; visual mesh filename=package://meshes/ef_body_1.stl scale=0.001 0.001 0.001
- added link left_gripper_1, mass 0.0035451260308642795; collision mesh filename=package://meshes/left_gripper_1.stl scale=0.001 0.001 0.001; visual mesh filename=package://meshes/left_gripper_1.stl scale=0.001 0.001 0.001
- added link right_gripper_1, mass 0.0035451260306269467; collision mesh filename=package://meshes/right_gripper_1.stl scale=0.001 0.001 0.001; visual mesh filename=package://meshes/right_gripper_1.stl scale=0.001 0.001 0.001
- link base_link: mass None -> 48.78806525610532
- link link_five_1: mass None -> 4.291162754920929
- link link_four_1: mass None -> 10.410422726556684
- link link_one_1: mass None -> 24.076192117313017
- link link_six_1: mass None -> 0.10737560006286881
- link link_three_1: mass None -> 23.108195954813556
- link link_two_1: mass None -> 30.683386891011434
Joints:
- added joint Rigid 10: type fixed, parent link_five_1, child camera_1, origin xyz=0.03103 0.040973 -0.00902 rpy=0 0 0
- added joint Rigid 11: type fixed, parent link_six_1, child ef_body_1, origin xyz=1e-06 2e-06 0.007 rpy=0 0 0
- added joint Rigid 8: type fixed, parent ef_body_1, child left_gripper_1, origin xyz=0.627907 -0.000127 0.442487 rpy=0 0 0
- added joint Rigid 9: type fixed, parent ef_body_1, child right_gripper_1, origin xyz=0.627907 -0.000127 0.442487 rpy=0 0 0
- joint Revolute 1: axis 0 -1 0 -> -0.0 -1.0 -0.0
- joint Revolute 2: axis -1 0 0 -> -1.0 0.0 0.000133
- joint Revolute 3: axis -1 0 0 -> -1.0 0.0 0.000133
- joint Revolute 4: axis 0 0 1 -> 0.000133 -0.000634 1.0
- joint Revolute 5: axis 1 0 0 -> 1.0 -0.000752 -0.000133
- joint Revolute 6: axis 0 0 1 -> 0.000134 0.000374 1.0
